File: discrete7segment.sch (KiCad schematic (older format))
At the start: 76 parts, among them P1 CONN_01X02, Q1 Q_NPN_BEC, Q2 Q_NPN_BEC, Q3 Q_NPN_BEC, Q4 Q_NPN_BEC, Q5 Q_NPN_BEC, Q6 Q_NPN_BEC, Q7 Q_NPN_BEC, U1 555, U2 4017

Commit message: layout begun
Parts:
- C1: footprint (none) -> Capacitors_SMD:C_1206_HandSoldering
- D1, D10, D11, D12, D13, D14, D15, D16, D17, D18, D19, D2, D20, D21, D22, D23, D24, D25, D26, D27, D28, D29, D3, D30, D31, D32, D33, D34, D35, D36, D37, D38, D39, D4, D40, D41, D42, D43, D44, D45, D46, D47, D48, D49, D5, D6, D7, D8, D9: footprint (none) -> Diodes_SMD:MiniMELF_Handsoldering
- D50, D51, D52, D53, D54, D55, D56, D57, D58, D59, D60, D61, D62, D63: footprint (none) -> LEDs:LED_0805
- P1: footprint (none) -> Pin_Headers:Pin_Header_Straight_1x02
- Q1, Q2, Q3, Q4, Q5, Q6, Q7: footprint (none) -> TO_SOT_Packages_SMD:SOT-23_Handsoldering
- R1, R2: footprint (none) -> Resistors_SMD:R_0805_HandSoldering
- U1: footprint (none) -> SMD_Packages:SOIC-8-N
- U2: footprint (none) -> SMD_Packages:SO-16-N

Commit message: generated schematic pdf
Other:
- note added: "Single digit\n7 segment display\nfrom discrete LEDs\nThe power is voltage-limited\nto <10mA so there's no need\nfor resistor(s)\n(EEs will disagree)"
- note removed: "Add resistor\nTypical voltage to drop will be 2.2V for each LED\nso there's not much to do, just limit current.\n>10mA suggested.\nAnd rewire transistors"
- note removed: "Single digit\n7 segment display\nfrom discrete LEDs"
Changed lines of the file:
@@
 This is a diode ROM\nsimilar that was used in pioneers of\ncomputing. Look up "diode matrix"
 Text Notes 9650 2350 0    60   ~ 0
-Single digit\n7 segment display\nfrom discrete LEDs
+Single digit\n7 segment display\nfrom discrete LEDs\nThe power is voltage-limited\nto <10mA so there's no need\nfor resistor(s)\n(EEs will disagree)
 Text Notes 5900 2550 0    60   ~ 0
 ROM -\nrows are digits\ncolumns are segments
@@
 $EndComp
 Connection ~ 10700 5800
-Text Notes 7600 6600 0    100  ~ 0
-Add resistor\nTypical voltage to drop will be 2.2V for each LED\nso there's not much to do, just limit current.\n>10mA suggested.\nAnd rewire transistors
 Text Notes 1300 6900 0    60   ~ 0
 Q: lolwtf?\nA: The matrix of diodes is hardwired memory.\n   Each row is one word/byte with the \n   length of 7 bits. The circuit 'stores' data\n   for displaying a number on a 7 segment LED display\n   (hence 7 bit word)\n   I'll be making the memory and the display from\n   discrete diodes and the only chips are for\n   changing the address. Counting up at 1Hz frequency.\n   It would also work by putting logic HIGH on anode\n   of one of the leftmost diodes and get your output\n   on the bottom. That's where the display is wired.

Commit message: found bugs, needs rework
Other:
- note added: "It's\nbuggy\nrewiring\nis\nnecessary"
Changed lines of the file:
@@
 Text Notes 1300 6900 0    60   ~ 0
 Q: lolwtf?\nA: The matrix of diodes is hardwired memory.\n   Each row is one word/byte with the \n   length of 7 bits. The circuit 'stores' data\n   for displaying a number on a 7 segment LED display\n   (hence 7 bit word)\n   I'll be making the memory and the display from\n   discrete diodes and the only chips are for\n   changing the address. Counting up at 1Hz frequency.\n   It would also work by putting logic HIGH on anode\n   of one of the leftmost diodes and get your output\n   on the bottom. That's where the display is wired.
+Text Notes 4550 5800 0    400  ~ 80
+It's\nbuggy\nrewiring\nis\nnecessary
 $EndSCHEMATC

Commit message: bugfixes
Connections:
- net b: now also D39.1 (K)
- net c: now also D47.1 (K)
- net e: no longer D34.1 (K)
- net f: now also D34.1 (K); no longer D39.1 (K)
- net g: no longer D47.1 (K)
Other:
- note added: "diode is 1\nno diode is 0"
- note removed: "It's\nbuggy\nrewiring\nis\nnecessary"
- moved on the sheet: D34, D39, D47
Changed lines of the file:
@@
 L D D47
 U 1 1 5ADB8642
-P 7150 4600
-F 0 "D47" H 7150 4700 50  0000 C CNN
-F 1 "D" H 7150 4500 50  0000 C CNN
-F 2 "Diodes_SMD:MiniMELF_Handsoldering" H 7150 4600 50  0001 C CNN
-F 3 "" H 7150 4600 50  0000 C CNN
-	1    7150 4600
+P 5550 4600
+F 0 "D47" H 5550 4700 50  0000 C CNN
+F 1 "D" H 5550 4500 50  0000 C CNN
+F 2 "Diodes_SMD:MiniMELF_Handsoldering" H 5550 4600 50  0001 C CNN
+F 3 "" H 5550 4600 50  0000 C CNN
+	1    5550 4600
 	-1   0    0    1
 $EndComp
@@
 L D D39
 U 1 1 5ADB86D0
-P 6750 4600
-F 0 "D39" H 6750 4700 50  0000 C CNN
-F 1 "D" H 6750 4500 50  0000 C CNN
-F 2 "Diodes_SMD:MiniMELF_Handsoldering" H 6750 4600 50  0001 C CNN
-F 3 "" H 6750 4600 50  0000 C CNN
-	1    6750 4600
+P 5150 4600
+F 0 "D39" H 5150 4700 50  0000 C CNN
+F 1 "D" H 5150 4500 50  0000 C CNN
+F 2 "Diodes_SMD:MiniMELF_Handsoldering" H 5150 4600 50  0001 C CNN
+F 3 "" H 5150 4600 50  0000 C CNN
+	1    5150 4600
 	-1   0    0    1
 $EndComp
@@
 L D D34
 U 1 1 5ADB8AAD
-P 6350 5300
-F 0 "D34" H 6350 5400 50  0000 C CNN
-F 1 "D" H 6350 5200 50  0000 C CNN
-F 2 "Diodes_SMD:MiniMELF_Handsoldering" H 6350 5300 50  0001 C CNN
-F 3 "" H 6350 5300 50  0000 C CNN
-	1    6350 5300
+P 6750 5300
+F 0 "D34" H 6750 5400 50  0000 C CNN
+F 1 "D" H 6750 5200 50  0000 C CNN
+F 2 "Diodes_SMD:MiniMELF_Handsoldering" H 6750 5300 50  0001 C CNN
+F 3 "" H 6750 5300 50  0000 C CNN
+	1    6750 5300
 	-1   0    0    1
 $EndComp
@@
 Text Notes 9650 2350 0    60   ~ 0
 Single digit\n7 segment display\nfrom discrete LEDs\nThe power is voltage-limited\nto <10mA so there's no need\nfor resistor(s)\n(EEs will disagree)
-Text Notes 5900 2550 0    60   ~ 0
+Text Notes 5850 2550 0    60   ~ 0
 ROM -\nrows are digits\ncolumns are segments
 Text Notes 4800 1300 0    60   ~ 0
 ! WARNING !\nThis circuit is not physically checked \nit would be a pain to put all on \nbreadboard but a perfboard might \nbe a relatively ok
-Text Notes 7300 1600 0    60   ~ 0
+Text Notes 7500 1800 0    60   ~ 0
   --a--\n|        |\nf         b\n|        |\n --g--\n|        |\ne        c\n|        |\n --d--
 $Comp
@@
 Connection ~ 6100 4200
 Connection ~ 6500 4200
-Connection ~ 6900 4600
 Connection ~ 6900 4200
 Connection ~ 6900 3800
@@
 Connection ~ 4900 4200
 Connection ~ 7300 4200
-Connection ~ 7300 4600
 Connection ~ 7300 4900
 Connection ~ 7300 5300
@@
 Connection ~ 6900 4900
 Connection ~ 6500 4900
-Connection ~ 6500 5300
+Connection ~ 6900 5300
 Connection ~ 6500 5600
 Connection ~ 6100 5300
@@
 Wire Wire Line
 	4600 5600 4600 5500
-Connection ~ 6200 5200
+Connection ~ 6600 5200
 Wire Wire Line
 	7000 5200 7000 5300
 Connection ~ 5800 5200
-Wire Wire Line
-	6200 5200 6200 5300
 Connection ~ 5400 5200
 Wire Wire Line
@@
 Wire Wire Line
 	4600 4900 4600 4800
-Connection ~ 6600 4500
-Wire Wire Line
-	7000 4500 7000 4600
-Wire Wire Line
-	6600 4500 6600 4600
-Wire Wire Line
-	4600 4500 7000 4500
 Wire Wire Line
 	4600 4600 4600 4500
@@
 	10700 5800 10500 5800
 Connection ~ 10700 5300
-Text Notes 8400 1700 0    60   ~ 0
+Text Notes 8600 1850 0    60   ~ 0
      abcdefg\n1 - 0110000\n2 - 1101101\n3 - 1111001\n4 - 0110011\n5 - 1011011\n6 - 1011111\n7 - 1110000\n8 - 1111111\n9 - 1111011\n0 - 1111110
 $Comp
@@
 Text Notes 1300 6900 0    60   ~ 0
 Q: lolwtf?\nA: The matrix of diodes is hardwired memory.\n   Each row is one word/byte with the \n   length of 7 bits. The circuit 'stores' data\n   for displaying a number on a 7 segment LED display\n   (hence 7 bit word)\n   I'll be making the memory and the display from\n   discrete diodes and the only chips are for\n   changing the address. Counting up at 1Hz frequency.\n   It would also work by putting logic HIGH on anode\n   of one of the leftmost diodes and get your output\n   on the bottom. That's where the display is wired.
-Text Notes 4550 5800 0    400  ~ 80
-It's\nbuggy\nrewiring\nis\nnecessary
+Text Notes 7000 2550 0    60   ~ 0
+diode is 1\nno diode is 0
+Wire Wire Line
+	4600 4500 5400 4500
+Wire Wire Line
+	5400 4500 5400 4600
+Wire Wire Line
+	5000 4500 5000 4600
+Connection ~ 5000 4500
+Connection ~ 5700 4600
+Connection ~ 5300 4600
+Wire Wire Line
+	6600 5200 6600 5300
 $EndSCHEMATC

Commit message: layout finished
Parts:
- D1, D10, D11, D12, D2, D3, D4, D40, D48, D49, D5, D6, D7, D8, D9: footprint Diodes_SMD:MiniMELF_Handsoldering -> Diodes_SMD:MiniMELF_Standard
- D13: renamed from D39; footprint Diodes_SMD:MiniMELF_Handsoldering -> Diodes_SMD:MiniMELF_Standard
- D14: renamed from D13; footprint Diodes_SMD:MiniMELF_Handsoldering -> Diodes_SMD:MiniMELF_Standard
- D15: renamed from D14; footprint Diodes_SMD:MiniMELF_Handsoldering -> Diodes_SMD:MiniMELF_Standard
- D16: renamed from D15; footprint Diodes_SMD:MiniMELF_Handsoldering -> Diodes_SMD:MiniMELF_Standard
- D17: renamed from D16; footprint Diodes_SMD:MiniMELF_Handsoldering -> Diodes_SMD:MiniMELF_Standard
- D18: renamed from D17; footprint Diodes_SMD:MiniMELF_Handsoldering -> Diodes_SMD:MiniMELF_Standard
- D19: renamed from D18; footprint Diodes_SMD:MiniMELF_Handsoldering -> Diodes_SMD:MiniMELF_Standard
- D20: renamed from D19; footprint Diodes_SMD:MiniMELF_Handsoldering -> Diodes_SMD:MiniMELF_Standard
- D21: renamed from D20; footprint Diodes_SMD:MiniMELF_Handsoldering -> Diodes_SMD:MiniMELF_Standard
- D22: renamed from D47; footprint Diodes_SMD:MiniMELF_Handsoldering -> Diodes_SMD:MiniMELF_Standard
- D23: renamed from D21; footprint Diodes_SMD:MiniMELF_Handsoldering -> Diodes_SMD:MiniMELF_Standard
- D24: renamed from D22; footprint Diodes_SMD:MiniMELF_Handsoldering -> Diodes_SMD:MiniMELF_Standard
- D25: renamed from D23; footprint Diodes_SMD:MiniMELF_Handsoldering -> Diodes_SMD:MiniMELF_Standard
- D26: renamed from D24; footprint Diodes_SMD:MiniMELF_Handsoldering -> Diodes_SMD:MiniMELF_Standard
- D27: renamed from D25; footprint Diodes_SMD:MiniMELF_Handsoldering -> Diodes_SMD:MiniMELF_Standard
- D28: renamed from D26; footprint Diodes_SMD:MiniMELF_Handsoldering -> Diodes_SMD:MiniMELF_Standard
- D29: renamed from D27; footprint Diodes_SMD:MiniMELF_Handsoldering -> Diodes_SMD:MiniMELF_Standard
- D30: renamed from D28; footprint Diodes_SMD:MiniMELF_Handsoldering -> Diodes_SMD:MiniMELF_Standard
- D31: renamed from D29; footprint Diodes_SMD:MiniMELF_Handsoldering -> Diodes_SMD:MiniMELF_Standard
- D32: renamed from D30; footprint Diodes_SMD:MiniMELF_Handsoldering -> Diodes_SMD:MiniMELF_Standard
- D33: renamed from D31; footprint Diodes_SMD:MiniMELF_Handsoldering -> Diodes_SMD:MiniMELF_Standard
- D34: renamed from D32; footprint Diodes_SMD:MiniMELF_Handsoldering -> Diodes_SMD:MiniMELF_Standard
- D35: renamed from D33; footprint Diodes_SMD:MiniMELF_Handsoldering -> Diodes_SMD:MiniMELF_Standard
- D36: renamed from D35; footprint Diodes_SMD:MiniMELF_Handsoldering -> Diodes_SMD:MiniMELF_Standard
- D37: renamed from D36; footprint Diodes_SMD:MiniMELF_Handsoldering -> Diodes_SMD:MiniMELF_Standard
- D38: renamed from D37; footprint Diodes_SMD:MiniMELF_Handsoldering -> Diodes_SMD:MiniMELF_Standard
- D39: renamed from D38; footprint Diodes_SMD:MiniMELF_Handsoldering -> Diodes_SMD:MiniMELF_Standard
- D41: renamed from D34; footprint Diodes_SMD:MiniMELF_Handsoldering -> Diodes_SMD:MiniMELF_Standard
- D42: renamed from D41; footprint Diodes_SMD:MiniMELF_Handsoldering -> Diodes_SMD:MiniMELF_Standard
- D43: renamed from D42; footprint Diodes_SMD:MiniMELF_Handsoldering -> Diodes_SMD:MiniMELF_Standard
- D44: renamed from D43; footprint Diodes_SMD:MiniMELF_Handsoldering -> Diodes_SMD:MiniMELF_Standard
- D45: renamed from D44; footprint Diodes_SMD:MiniMELF_Handsoldering -> Diodes_SMD:MiniMELF_Standard
- D46: renamed from D45; footprint Diodes_SMD:MiniMELF_Handsoldering -> Diodes_SMD:MiniMELF_Standard
- D47: renamed from D46; footprint Diodes_SMD:MiniMELF_Handsoldering -> Diodes_SMD:MiniMELF_Standard

Commit message: bugfix
Parts:
- removed C1: 2.2uF, Capacitors_SMD:C_1206_HandSoldering, symbol CP1
- added C1: 2.2uF, symbol C
Connections:
- net GND: now also C1.2; no longer U1.5 (CTRL)
- net at R2.2 (K), U1.2 (TRIG), U1.6 (THR): now also C1.1
- no-connect marks 1 -> 2
Changed lines of the file:
@@
   --a--\n|        |\nf         b\n|        |\n --g--\n|        |\ne        c\n|        |\n --d--
 $Comp
-L PWR_FLAG #FLG01
+L PWR_FLAG #FLG1
 U 1 1 5ADB9598
 P 3550 1250
-F 0 "#FLG01" H 3550 1345 50  0001 C CNN
+F 0 "#FLG1" H 3550 1345 50  0001 C CNN
 F 1 "PWR_FLAG" H 3550 1430 50  0000 C CNN
 F 2 "" H 3550 1250 50  0000 C CNN
@@
 $EndComp
 $Comp
-L PWR_FLAG #FLG02
+L PWR_FLAG #FLG2
 U 1 1 5ADB96EF
 P 3550 1450
-F 0 "#FLG02" H 3550 1545 50  0001 C CNN
+F 0 "#FLG2" H 3550 1545 50  0001 C CNN
 F 1 "PWR_FLAG" H 3550 1630 50  0000 C CNN
 F 2 "" H 3550 1450 50  0000 C CNN
@@
 $EndComp
 $Comp
-L GND #PWR03
+L GND #PWR7
 U 1 1 5ADB9C02
 P 3850 1450
-F 0 "#PWR03" H 3850 1200 50  0001 C CNN
+F 0 "#PWR7" H 3850 1200 50  0001 C CNN
 F 1 "GND" H 3850 1300 50  0000 C CNN
 F 2 "" H 3850 1450 50  0000 C CNN
@@
 $EndComp
 $Comp
-L +5V #PWR04
+L +5V #PWR6
 U 1 1 5ADB9C9A
 P 3850 1250
-F 0 "#PWR04" H 3850 1100 50  0001 C CNN
+F 0 "#PWR6" H 3850 1100 50  0001 C CNN
 F 1 "+5V" H 3850 1390 50  0000 C CNN
 F 2 "" H 3850 1250 50  0000 C CNN
@@
 $EndComp
 $Comp
-L +5V #PWR05
+L +5V #PWR3
 U 1 1 5ADB9DB4
 P 2600 2150
-F 0 "#PWR05" H 2600 2000 50  0001 C CNN
+F 0 "#PWR3" H 2600 2000 50  0001 C CNN
 F 1 "+5V" H 2600 2290 50  0000 C CNN
 F 2 "" H 2600 2150 50  0000 C CNN
@@
 $EndComp
 $Comp
-L +5V #PWR06
+L +5V #PWR4
 U 1 1 5ADB9F4B
 P 2800 3950
-F 0 "#PWR06" H 2800 3800 50  0001 C CNN
+F 0 "#PWR4" H 2800 3800 50  0001 C CNN
 F 1 "+5V" H 2800 4090 50  0000 C CNN
 F 2 "" H 2800 3950 50  0000 C CNN
@@
 $EndComp
 $Comp
-L GND #PWR07
+L GND #PWR2
 U 1 1 5ADBA3CC
-P 2600 3450
-F 0 "#PWR07" H 2600 3200 50  0001 C CNN
-F 1 "GND" H 2600 3300 50  0000 C CNN
-F 2 "" H 2600 3450 50  0000 C CNN
-F 3 "" H 2600 3450 50  0000 C CNN
-	1    2600 3450
-	1    0    0    -1
-$EndComp
-$Comp
-L GND #PWR08
+P 2400 3450
+F 0 "#PWR2" H 2400 3200 50  0001 C CNN
+F 1 "GND" H 2400 3300 50  0000 C CNN
+F 2 "" H 2400 3450 50  0000 C CNN
+F 3 "" H 2400 3450 50  0000 C CNN
+	1    2400 3450
+	1    0    0    -1
+$EndComp
+$Comp
+L GND #PWR5
 U 1 1 5ADBA49D
 P 2800 5150
-F 0 "#PWR08" H 2800 4900 50  0001 C CNN
+F 0 "#PWR5" H 2800 4900 50  0001 C CNN
 F 1 "GND" H 2800 5000 50  0000 C CNN
 F 2 "" H 2800 5150 50  0000 C CNN
@@
 	3350 2800 3350 3800
 Wire Wire Line
-	1900 3450 2800 3450
-Connection ~ 2600 3450
-Wire Wire Line
 	1900 2150 2800 2150
 Connection ~ 2600 2150
@@
 Wire Wire Line
 	2050 3000 1900 3000
-$Comp
-L CP1 C1
-U 1 1 5ADC2A8C
-P 1900 3200
-F 0 "C1" H 1950 3300 50  0000 L CNN
-F 1 "2.2uF" H 1950 3100 50  0000 L CNN
-F 2 "Capacitors_SMD:C_1206_HandSoldering" H 1900 3200 60  0001 C CNN
-F 3 "" H 1900 3200 60  0000 C CNN
-	1    1900 3200
-	1    0    0    -1
-$EndComp
 Wire Wire Line
 	1900 3450 1900 3400
@@
 	2150 4100 2150 4450
 $Comp
-L GND #PWR09
+L GND #PWR1
 U 1 1 5ADC678C
 P 2150 4450
-F 0 "#PWR09" H 2150 4200 50  0001 C CNN
+F 0 "#PWR1" H 2150 4200 50  0001 C CNN
 F 1 "GND" H 2150 4300 50  0000 C CNN
 F 2 "" H 2150 4450 50  0000 C CNN
@@
 $EndComp
 $Comp
-L +5V #PWR010
+L +5V #PWR8
 U 1 1 5ADCE83C
 P 9200 2300
-F 0 "#PWR010" H 9200 2150 50  0001 C CNN
+F 0 "#PWR8" H 9200 2150 50  0001 C CNN
 F 1 "+5V" H 9200 2440 50  0000 C CNN
 F 2 "" H 9200 2300 50  0000 C CNN
@@
      abcdefg\n1 - 0110000\n2 - 1101101\n3 - 1111001\n4 - 0110011\n5 - 1011011\n6 - 1011111\n7 - 1110000\n8 - 1111111\n9 - 1111011\n0 - 1111110
 $Comp
-L GND #PWR011
+L GND #PWR9
 U 1 1 5ADDC501
 P 10700 5900
-F 0 "#PWR011" H 10700 5650 50  0001 C CNN
+F 0 "#PWR9" H 10700 5650 50  0001 C CNN
 F 1 "GND" H 10700 5750 50  0000 C CNN
 F 2 "" H 10700 5900 50  0000 C CNN
@@
 Wire Wire Line
 	6600 5200 6600 5300
+Wire Wire Line
+	2400 3450 1900 3450
+NoConn ~ 2800 3450
+$Comp
+L C C1
+U 1 1 5AF40DAE
+P 1900 3200
+F 0 "C1" H 1900 3300 40  0000 L CNN
+F 1 "2.2uF" H 1906 3115 40  0000 L CNN
+F 2 "" H 1938 3050 30  0000 C CNN
+F 3 "" H 1900 3200 60  0000 C CNN
+	1    1900 3200
+	1    0    0    -1
+$EndComp
+Connection ~ 1900 3000
 $EndSCHEMATC

Commit message: details
Other:
- note removed: "! WARNING !\nThis circuit is not physically checked \nit would be a pain to put all on \nbreadboard but a perfboard might \nbe a relatively ok"
Changed lines of the file:
@@
 Text Notes 5850 2550 0    60   ~ 0
 ROM -\nrows are digits\ncolumns are segments
-Text Notes 4800 1300 0    60   ~ 0
-! WARNING !\nThis circuit is not physically checked \nit would be a pain to put all on \nbreadboard but a perfboard might \nbe a relatively ok
 Text Notes 7500 1800 0    60   ~ 0
   --a--\n|        |\nf         b\n|        |\n --g--\n|        |\ne        c\n|        |\n --d--

Commit message: vast redesign
Parts:
- removed D50, D51, D52, D53, D54, D55, D56, D57, D58, D59, D60, D61, D62, D63: LED, LEDs:LED_0805, symbol LED
- removed Q1, Q2, Q3, Q4, Q5, Q6, Q7: Q_NPN_BEC, TO_SOT_Packages_SMD:SOT-23_Handsoldering, symbol Q_NPN_BEC
- added C2: 1uF, symbol C
- added P2: CLK, symbol CONN_01X01
- added P3: CONN_01X10, symbol CONN_01X10
- added Q1, Q2, Q3, Q4, Q5, Q6, Q7: Q_NPN_CBE, symbol Q_NPN_CBE
- added R3, R4, R5, R6, R7, R8, R9: 330, symbol R
- added SW1: SPDT, symbol SPDT
- added U3: 78L05, symbol 78L05
- added U4: 7-seg_1-dig, symbol 7-seg_1-dig
Connections:
- net +5V: now also Q1.1 (C), Q2.1 (C), Q3.1 (C), Q4.1 (C), Q5.1 (C), Q6.1 (C), Q7.1 (C), U3.1 (OUT); no longer P1.1 (P1)
- net GND: now also C2.2, U3.2 (GND), U4.3 (GND), U4.8 (GND)
- net a: now also Q1.2 (B)
- net b: now also Q2.2 (B)
- net c: now also Q3.2 (B)
- net d: now also Q4.2 (B)
- net e: now also Q5.2 (B)
- net f: now also Q6.2 (B)
- net g: now also Q7.2 (B)
- net 6: now reaches D21.2 (A), D29.2 (A), D34.2 (A), D39.2 (A), D4.2 (A), D47.2 (A), U2.1 (Q5)
- net 6: now also P3.6 (P6)
- net 5: now reaches D20.2 (A), D28.2 (A), D3.2 (A), D38.2 (A), D46.2 (A), U2.10 (Q4)
- net 5: now also P3.5 (P5)
- net 0: now reaches D16.2 (A), D25.2 (A), D32.2 (A), D36.2 (A), D42.2 (A), D8.2 (A), U2.11 (Q9)
- net 0: now also P3.10 (P10)
- net at U2.14 (CLK): now also P2.1 (P1), SW1.2; no longer U1.3 (OUT)
- net 2: now reaches D1.2 (A), D10.2 (A), D26.2 (A), D33.2 (A), D43.2 (A), U2.2 (Q1)
- net 2: now also P3.2 (P2)
- net 1: now reaches D17.2 (A), D9.2 (A), U2.3 (Q0)
- net 1: now also P3.1 (P1)
- net 3: now reaches D11.2 (A), D18.2 (A), D2.2 (A), D27.2 (A), D44.2 (A), U2.4 (Q2)
- net 3: now also P3.3 (P3)
- net 7: now reaches D13.2 (A), D22.2 (A), D5.2 (A), U2.5 (Q6)
- net 7: now also P3.7 (P7)
- net 8: now reaches D14.2 (A), D23.2 (A), D30.2 (A), D35.2 (A), D40.2 (A), D48.2 (A), D6.2 (A), U2.6 (Q7)
- net 8: now also P3.8 (P8)
- net 4: now reaches D12.2 (A), D19.2 (A), D37.2 (A), D45.2 (A), U2.7 (Q3)
- net 4: now also P3.4 (P4)
- net 9: now reaches D15.2 (A), D24.2 (A), D31.2 (A), D41.2 (A), D49.2 (A), D7.2 (A), U2.9 (Q8)
- net 9: now also P3.9 (P9)
- new net: C2.1, P1.1 (P1), U3.3 (IN)
- new net: SW1.1, U1.3 (OUT)
- new net: R7.2 (K), U4.1 (E)
- new net: R9.2 (K), U4.10 (G)
- new net: R6.2 (K), U4.2 (D)
- new net: R5.2 (K), U4.4 (C)
- new net: R4.2 (K), U4.6 (B)
- new net: R3.2 (K), U4.7 (A)
- new net: R8.2 (K), U4.9 (F)
- new net: Q1.3 (E), R3.1 (A)
- new net: Q2.3 (E), R4.1 (A)
- new net: Q3.3 (E), R5.1 (A)
- new net: Q4.3 (E), R6.1 (A)
- new net: Q5.3 (E), R7.1 (A)
- new net: Q6.3 (E), R8.1 (A)
- new net: Q7.3 (E), R9.1 (A)
- no-connect marks 2 -> 4
Other:
- note added: "1.7V drop per segment"
- note added: "Aiming for 10mA per\nsegment"
- note added: "BC547"
- note added: "Direct\naccess\npin\nheadder"
- note added: "Manual\nclock"
- note added: "Rows are digits, columns are segments"
- note added: "orange\norange\nbrown"
- note removed: "1\n\n\n2\n\n\n3\n\n\n4\n\n\n5\n\n\n6\n\n\n7\n\n\n8\n\n\n9\n\n\n0"
- note removed: "ROM -\nrows are digits\ncolumns are segments"
- note removed: "Single digit\n7 segment display\nfrom discrete LEDs\nThe power is voltage-limited\nto <10mA so there's no need\nfor resistor(s)\n(EEs will disagree)"
- note removed: "a b c d e f g"
- moved on the sheet: C1, D1, D10, D11, D12, D13, D14, D15, D16, D17, D18, D19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
