File: discrete7segment.kicad_pcb (KiCad board)
At the start: 2 copper layers, 99.1 x 76.2 mm, 75 parts, among them P1 CONN_01X02, P2 CLK, P3 CONN_01X10, Q1 Q_NPN_CBE, Q2 Q_NPN_CBE, Q3 Q_NPN_CBE, Q4 Q_NPN_CBE, Q5 Q_NPN_CBE, Q6 Q_NPN_CBE, Q7 Q_NPN_CBE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

Commit message: erc passed
Routing:
- net +5V: track 111.3 -> 150.8 mm
- net GND: track 0.00 -> 14.8 mm, vias 0 -> 2
- net Net-(C2-Pad1): track 19.9 -> 9.04 mm
- net /c: track 53.9 -> 64.0 mm
- added copper zone on F.Cu, net Net-(C2-Pad1)
Other:
- board text added: "05/18 Rev2"
- board text added: "1uF"
- board text added: "2.2uF"
- board text removed: "05/18"
Changed lines of the file:
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@@
   (general
     (links 152)
-    (no_connects 6)
+    (no_connects 0)
     (area 68.504999 86.284999 167.715001 162.635001)
     (thickness 1.6)
-    (drawings 23)
-    (tracks 428)
+    (drawings 25)
+    (tracks 453)
     (zones 0)
     (modules 75)
@@
     (pad_to_mask_clearance 0.2)
     (aux_axis_origin 0 0)
-    (visible_elements FFFFF77F)
+    (grid_origin 68.58 86.36)
+    (visible_elements FFFFFF7F)
     (pcbplotparams
       (layerselection 0x030f0_80000001)
@@
       (net 37 "Net-(R9-Pad2)"))
   )
-  (gr_text 05/18 (at 163.83 161.29) (layer F.SilkS)
+  (gr_text 2.2uF (at 73.66 101.6 90) (layer F.SilkS)
+    (effects (font (size 0.889 0.889) (thickness 0.22225)))
+  )
+  (gr_text 1uF (at 73.66 93.98 90) (layer F.SilkS)
+    (effects (font (size 0.889 0.889) (thickness 0.22225)))
+  )
+  (gr_text "05/18 Rev2" (at 160.02 161.29) (layer F.SilkS)
     (effects (font (size 1.5 1.5) (thickness 0.3)))
   )
@@
     (effects (font (size 2.54 2.54) (thickness 0.508)))
   )
-  (gr_text "Unregulated Powersupply" (at 91.44 158.75) (layer F.SilkS)
+  (gr_text "Unregulated Powersupply" (at 88.9 158.75) (layer F.SilkS)
     (effects (font (size 1.778 1.778) (thickness 0.3)))
   )
@@
     (effects (font (size 1.5 1.5) (thickness 0.3)))
   )
-  (gr_text 78L05 (at 83.82 88.9 90) (layer F.SilkS)
+  (gr_text 78L05 (at 87.63 86.995) (layer F.SilkS)
     (effects (font (size 0.889 0.889) (thickness 0.22225)))
   )
@@
   (segment (start 91.44 101.6) (end 86.36 101.6) (width 0.25) (layer F.Cu) (net 1))
   (segment (start 86.36 101.6) (end 83.82 99.06) (width 0.25) (layer F.Cu) (net 1))
+  (segment (start 83.82 132.08) (end 85.09 132.08) (width 0.25) (layer B.Cu) (net 2))
+  (segment (start 90.17 121.92) (end 91.44 121.92) (width 0.25) (layer B.Cu) (net 2))
+  (segment (start 89.535 122.555) (end 90.17 121.92) (width 0.25) (layer B.Cu) (net 2))
+  (via (at 89.535 122.555) (size 0.6) (drill 0.4) (layers F.Cu B.Cu) (net 2))
+  (segment (start 89.535 127.635) (end 89.535 122.555) (width 0.25) (layer F.Cu) (net 2))
+  (segment (start 88.9 128.27) (end 89.535 127.635) (width 0.25) (layer F.Cu) (net 2))
+  (via (at 88.9 128.27) (size 0.6) (drill 0.4) (layers F.Cu B.Cu) (net 2))
+  (segment (start 85.09 132.08) (end 88.9 128.27) (width 0.25) (layer B.Cu) (net 2))
   (segment (start 116.84 134.62) (end 116.84 139.7) (width 0.25) (layer B.Cu) (net 3))
   (segment (start 115.57 140.97) (end 115.57 142.24) (width 0.25) (layer B.Cu) (net 3))
@@
   (segment (start 124.46 139.7) (end 124.46 134.62) (width 0.25) (layer B.Cu) (net 4))
   (segment (start 123.19 140.97) (end 124.46 139.7) (width 0.25) (layer B.Cu) (net 4))
+  (segment (start 132.08 104.14) (end 132.08 109.22) (width 0.25) (layer B.Cu) (net 5))
+  (segment (start 132.08 119.38) (end 132.08 124.46) (width 0.25) (layer B.Cu) (net 5))
   (segment (start 132.08 134.62) (end 132.08 139.7) (width 0.25) (layer B.Cu) (net 5))
   (segment (start 130.81 140.97) (end 130.81 142.24) (width 0.25) (layer B.Cu) (net 5))
@@
   (segment (start 162.56 99.06) (end 162.56 104.14) (width 0.25) (layer B.Cu) (net 9))
   (segment (start 162.56 93.98) (end 162.56 99.06) (width 0.25) (layer B.Cu) (net 9))
+  (segment (start 154.94 142.24) (end 154.94 143.51) (width 0.25) (layer B.Cu) (net 10))
+  (segment (start 154.94 143.51) (end 156.21 144.78) (width 0.25) (layer B.Cu) (net 10))
+  (segment (start 153.67 144.78) (end 154.94 143.51) (width 0.25) (layer B.Cu) (net 10))
+  (segment (start 154.94 142.24) (end 154.94 143.51) (width 0.25) (layer B.Cu) (net 10))
+  (segment (start 154.94 143.51) (end 154.94 142.24) (width 0.25) (layer B.Cu) (net 10))
+  (segment (start 78.74 109.22) (end 83.82 109.22) (width 0.25) (layer B.Cu) (net 10))
+  (segment (start 88.9 114.3) (end 91.44 114.3) (width 0.25) (layer B.Cu) (net 10))
+  (segment (start 83.82 109.22) (end 88.9 114.3) (width 0.25) (layer B.Cu) (net 10))
+  (segment (start 83.82 104.14) (end 78.74 109.22) (width 0.25) (layer B.Cu) (net 10))
+  (segment (start 91.44 96.52) (end 90.805 96.52) (width 0.25) (layer B.Cu) (net 10))
+  (segment (start 90.805 96.52) (end 86.995 100.33) (width 0.25) (layer B.Cu) (net 10))
+  (segment (start 86.995 100.33) (end 86.995 103.505) (width 0.25) (layer B.Cu) (net 10))
+  (segment (start 86.995 103.505) (end 86.36 104.14) (width 0.25) (layer B.Cu) (net 10))
+  (segment (start 86.36 104.14) (end 83.82 104.14) (width 0.25) (layer B.Cu) (net 10))
   (segment (start 116.84 142.24) (end 116.84 143.51) (width 0.25) (layer B.Cu) (net 10))
   (segment (start 116.84 143.51) (end 115.57 144.78) (width 0.25) (layer B.Cu) (net 10))
+  (segment (start 115.57 144.78) (end 105.41 144.78) (width 0.25) (layer B.Cu) (net 10))
+  (segment (start 105.41 144.78) (end 100.33 139.7) (width 0.25) (layer B.Cu) (net 10))
+  (segment (start 100.33 139.7) (end 100.33 115.57) (width 0.25) (layer B.Cu) (net 10))
+  (segment (start 100.33 115.57) (end 99.06 114.3) (width 0.25) (layer B.Cu) (net 10))
   (segment (start 99.06 114.3) (end 91.44 114.3) (width 0.25) (layer B.Cu) (net 10))
-  (segment (start 100.33 115.57) (end 99.06 114.3) (width 0.25) (layer B.Cu) (net 10))
-  (segment (start 100.33 139.7) (end 100.33 115.57) (width 0.25) (layer B.Cu) (net 10))
-  (segment (start 105.41 144.78) (end 100.33 139.7) (width 0.25) (layer B.Cu) (net 10))
-  (segment (start 115.57 144.78) (end 105.41 144.78) (width 0.25) (layer B.Cu) (net 10))
   (segment (start 147.32 142.24) (end 147.32 143.51) (width 0.25) (layer B.Cu) (net 10))
   (segment (start 147.32 143.51) (end 148.59 144.78) (width 0.25) (layer B.Cu) (net 10))
   (segment (start 162.56 143.51) (end 162.56 142.24) (width 0.25) (layer B.Cu) (net 10))
   (segment (start 161.29 144.78) (end 162.56 143.51) (width 0.25) (layer B.Cu) (net 10))
-  (segment (start 148.59 144.78) (end 161.29 144.78) (width 0.25) (layer B.Cu) (net 10))
+  (segment (start 148.59 144.78) (end 153.67 144.78) (width 0.25) (layer B.Cu) (net 10))
+  (segment (start 156.21 144.78) (end 161.29 144.78) (width 0.25) (layer B.Cu) (net 10))
   (segment (start 139.7 142.24) (end 139.7 143.51) (width 0.25) (layer B.Cu) (net 10))
   (segment (start 139.7 143.51) (end 140.97 144.78) (width 0.25) (layer B.Cu) (net 10))
@@
   (segment (start 78.74 114.3) (end 85.09 107.95) (width 0.25) (layer F.Cu) (net 11))
   (segment (start 73.66 116.84) (end 78.74 116.84) (width 0.25) (layer F.Cu) (net 11))
-  (segment (start 76.2 93.98) (end 76.2 91.44) (width 0.25) (layer F.Cu) (net 12))
-  (segment (start 76.2 91.44) (end 78.74 88.9) (width 0.25) (layer F.Cu) (net 12))
-  (segment (start 78.74 88.9) (end 86.36 88.9) (width 0.25) (layer F.Cu) (net 12))
-  (segment (start 71.12 88.9) (end 73.66 88.9) (width 0.25) (layer F.Cu) (net 12))
-  (segment (start 73.66 88.9) (end 76.2 91.44) (width 0.25) (layer F.Cu) (net 12))
+  (segment (start 76.2 93.98) (end 74.295 93.98) (width 0.25) (layer F.Cu) (net 12))
+  (segment (start 72.39 88.9) (end 71.12 88.9) (width 0.25) (layer F.Cu) (net 12))
+  (segment (start 73.66 90.17) (end 72.39 88.9) (width 0.25) (layer F.Cu) (net 12))
+  (segment (start 73.66 93.345) (end 73.66 90.17) (width 0.25) (layer F.Cu) (net 12))
+  (segment (start 74.295 93.98) (end 73.66 93.345) (width 0.25) (layer F.Cu) (net 12))
   (segment (start 143.51 93.98) (end 143.51 92.71) (width 0.25) (layer F.Cu) (net 13))
   (segment (start 143.51 92.71) (end 144.78 91.44) (width 0.25) (layer F.Cu) (net 13))
@@
   (segment (start 76.2 109.22) (end 76.2 110.49) (width 0.25) (layer F.Cu) (net 38))
   (segment (start 80.01 105.41) (end 76.2 109.22) (width 0.25) (layer F.Cu) (net 38))
-  (zone (net 10) (net_name +5V) (layer F.Cu) (hatch edge 0.508)
-    (connect_pads (clearance 0.508))
-    (min_thickness 0.254)
-    (fill yes (arc_segments 16) (thermal_gap 0.508) (thermal_bridge_width 0.508))
-    (polygon
-      (pts
-        (xy 101.6 162.56) (xy 68.58 162.56) (xy 68.58 86.36) (xy 101.6 86.36)
-      )
-    )
-  )
   (zone (net 2) (net_name GND) (layer B.Cu) (hatch edge 0.508)
     (connect_pads (clearance 0.508))
@@
       )
     )
+  )
+  (zone (net 12) (net_name "Net-(C2-Pad1)") (layer F.Cu) (hatch edge 0.508)
+    (connect_pads (clearance 0.508))
+    (min_thickness 0.254)
+    (fill yes (arc_segments 16) (thermal_gap 0.508) (thermal_bridge_width 0.508))
+    (polygon
+      (pts
+        (xy 86.995 93.98) (xy 68.58 93.98) (xy 68.58 86.36) (xy 86.995 86.36)
+      )
+    )
+  )
+  (zone (net 10) (net_name +5V) (layer F.Cu) (hatch edge 0.508)
+    (connect_pads (clearance 0.508))
+    (min_thickness 0.254)
+    (fill yes (arc_segments 16) (thermal_gap 0.508) (thermal_bridge_width 0.508))
+    (polygon
+      (pts
+        (xy 101.6 162.56) (xy 68.58 162.56) (xy 68.58 95.25) (xy 88.265 95.25) (xy 88.265 86.36)
+        (xy 101.6 86.36)
+      )
+    )
